Commit message: change env parameters

File: env/data/peg_in_hole_board/board_easy.urdf (robot description, URDF)
Before this commit: robot board, 2 links, 1 joints
Joints:
- joint board__circle: origin xyz=0.0 0.190 0.0 rpy=0 0 0 -> xyz=0.0 0.20 0.0 rpy=0 0 0

File: env/data/peg_in_hole_board/board_hard.urdf (robot description, URDF)
Before this commit: robot board, 2 links, 1 joints
Joints:
- joint board__circle: origin xyz=0.0 0.190 0.0 rpy=0 0 0 -> xyz=0.0 0.20 0.0 rpy=0 0 0
